File: Eagle/RGBNDR.brd (EAGLE design)
At the start: 110 parts, among them Q1 2N2222, Q2 2N2222

Commit message: reset brd
Parts:
- moved G_IN 278.5 mm to (-109.2, 25.4)
- moved AMP_2_IN 270.3 mm to (-71.1, 8.89)
- moved B_IN 262.7 mm to (-97.8, 25.4)
- moved MODE_IN 238.7 mm to (-86.4, 41.9)
- moved ALL_IN 236.1 mm to (-74.9, 25.4)
- moved OSC_1_SYNC 233.8 mm to (-85.1, 7.62)
- moved AMP_1_IN 231.2 mm to (-36.8, 8.89)
- moved OSC_2_SYNC 229.6 mm to (-96.5, 7.62)
- moved OSC_3_SYNC 222.1 mm to (-108.0, 7.62)
- moved OSC_1_SQ 208.1 mm to (-109.2, 41.9)
- moved MIX_OUT 186.0 mm to (-74.9, 41.9)
- moved R_IN 183.4 mm to (-17.8, 69.8)
- moved MIX_IN_5 179.5 mm to (-63.5, 41.9)
- moved AMP_3_IN 176.1 mm to (-86.4, 25.4)
- moved MIX_IN_4 174.0 mm to (-52.1, 41.9)
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Other:
- board outline added: 160 x 100 mm
